Commit message: Rectify URDF to confirm TCP orientation

File: mec_arm_model/urdf/mec_arm.urdf (robot description, URDF)
Before this commit: robot mec_arm_6dof, 10 links, 9 joints
Links:
- added link TCP_link
Joints:
- added joint TCP_fixed_joint: type fixed, parent Empty_Link6, child TCP_link, origin xyz=0 0 0.20 rpy=0 0 -0.8724
